Commit message: replaced the robot with something very simple, to increase performance. added LIDAR and camera

File: robot_sim_sose/src/xgo_description/urdf/xgo.urdf (robot description, URDF)
Before this commit: robot xgo, 22 links, 21 joints
Links:
- removed link arm_calf
- removed link arm_thigh
- removed link base
- removed link bl_calf
- removed link bl_foot
- removed link bl_hip
- removed link bl_thigh
- removed link body
- removed link br_calf
- removed link br_foot
- removed link br_hip
- removed link br_thigh
- removed link fl_calf
- removed link fl_foot
- removed link fl_hip
- removed link fl_thigh
- removed link fr_calf
- removed link fr_foot
- removed link fr_hip
- removed link fr_thigh
- removed link hand_left
- removed link hand_right
- added link base_link, mass 2.0; collision box size=0.25 0.15 0.10; visual box size=0.25 0.15 0.10
- added link camera_link, mass 0.1; collision box size=0.04 0.04 0.03; visual box size=0.04 0.04 0.03
- added link front_left_wheel, mass 1.0; collision cylinder length=0.02 radius=0.05; visual cylinder length=0.02 radius=0.05
- added link front_right_wheel, mass 1.0; collision cylinder length=0.02 radius=0.05; visual cylinder length=0.02 radius=0.05
- added link lidar_link, mass 0.2; collision cylinder length=0.03 radius=0.04; visual cylinder length=0.03 radius=0.04
- added link rear_left_wheel, mass 1.0; collision cylinder length=0.02 radius=0.05; visual cylinder length=0.02 radius=0.05
- added link rear_right_wheel, mass 1.0; collision cylinder length=0.02 radius=0.05; visual cylinder length=0.02 radius=0.05
Joints:
- removed joint arm_calf_joint
- removed joint arm_thigh_joint
- removed joint bl_calf_joint
- removed joint bl_foot_joint
- removed joint bl_hip_joint
- removed joint bl_thigh_joint
- removed joint br_calf_joint
- removed joint br_foot_joint
- removed joint br_hip_joint
- removed joint br_thigh_joint
- removed joint fl_calf_joint
- removed joint fl_foot_joint
- removed joint fl_hip_joint
- removed joint fl_thigh_joint
- removed joint floating_base
- removed joint fr_calf_joint
- removed joint fr_foot_joint
- removed joint fr_hip_joint
- removed joint fr_thigh_joint
- removed joint hand_left_joint
- removed joint hand_right_joint
- added joint camera_joint: type fixed, parent base_link, child camera_link, origin xyz=0.14 0 0.10 rpy=0 0 0
- added joint front_left_wheel_joint: type continuous, parent base_link, child front_left_wheel, origin xyz=0.08 0.075 0.02 rpy=1.5707 0 0, axis 0 1 0
- added joint front_right_wheel_joint: type continuous, parent base_link, child front_right_wheel, origin xyz=0.08 -0.075 0.02 rpy=1.5707 0 0, axis 0 1 0
- added joint lidar_joint: type fixed, parent base_link, child lidar_link, origin xyz=0 0 0.12 rpy=0 0 0
- added joint rear_left_wheel_joint: type continuous, parent base_link, child rear_left_wheel, origin xyz=-0.08 0.075 0.02 rpy=1.5707 0 0, axis 0 1 0
- added joint rear_right_wheel_joint: type continuous, parent base_link, child rear_right_wheel, origin xyz=-0.08 -0.075 0.02 rpy=1.5707 0 0, axis 0 1 0

Commit message: added a dummy explore function, that moves forward and rotates. removed 2 wheels, to get the rotation working for now, need a better solution

File: robot_sim_sose/src/xgo_description/urdf/xgo.urdf (robot description, URDF)
Before this commit: robot xgo_simple, 7 links, 6 joints
Links:
- removed link rear_left_wheel
- removed link rear_right_wheel
Joints:
- removed joint rear_left_wheel_joint
- removed joint rear_right_wheel_joint
- joint front_left_wheel_joint: axis 0 1 0 -> 0 0 -1
- joint front_right_wheel_joint: axis 0 1 0 -> 0 0 -1

Commit message: updated the robots optics, 4 wheels, the main box isnt on the ground anymore and does not intersect with the wheels

File: robot_sim_sose/src/xgo_description/urdf/xgo.urdf (robot description, URDF)
Before this commit: robot xgo_simple, 5 links, 4 joints
Links:
- added link rear_left_wheel, mass 0.2; collision cylinder length=0.02 radius=0.05; visual cylinder length=0.02 radius=0.05
- added link rear_right_wheel, mass 0.2; collision cylinder length=0.02 radius=0.05; visual cylinder length=0.02 radius=0.05
- link front_left_wheel: mass 1.0 -> 0.2
- link front_right_wheel: mass 1.0 -> 0.2
Joints:
- added joint rear_left_wheel_joint: type continuous, parent base_link, child rear_left_wheel, origin xyz=-0.08 0.09 0.05 rpy=1.5707 0 0, axis 0 0 -1
- added joint rear_right_wheel_joint: type continuous, parent base_link, child rear_right_wheel, origin xyz=-0.08 -0.09 0.05 rpy=1.5707 0 0, axis 0 0 -1
- joint front_left_wheel_joint: origin xyz=0.08 0.075 0.02 rpy=1.5707 0 0 -> xyz=0.08 0.09 0.05 rpy=1.5707 0 0
- joint front_right_wheel_joint: origin xyz=0.08 -0.075 0.02 rpy=1.5707 0 0 -> xyz=0.08 -0.09 0.05 rpy=1.5707 0 0
- joint lidar_joint: origin xyz=0 0 0.12 rpy=0 0 0 -> xyz=0 0 0.15 rpy=0 0 0

Commit message: fixed movement problems with the robot

File: robot_sim_sose/src/xgo_description/urdf/xgo.urdf (robot description, URDF)
Before this commit: robot xgo_simple, 7 links, 6 joints
Links:
- added link middle_left_wheel, mass 0.2; collision cylinder length=0.02 radius=0.05; visual cylinder length=0.02 radius=0.05
- added link middle_right_wheel, mass 0.2; collision cylinder length=0.02 radius=0.05; visual cylinder length=0.02 radius=0.05
Joints:
- added joint middle_left_wheel_joint: type continuous, parent base_link, child middle_left_wheel, origin xyz=0.00 0.09 0.05 rpy=1.5707 0 0, axis 0 0 -1
- added joint middle_right_wheel_joint: type continuous, parent base_link, child middle_right_wheel, origin xyz=0.00 -0.09 0.05 rpy=1.5707 0 0, axis 0 0 -1
- joint front_left_wheel_joint: origin xyz=0.08 0.09 0.05 rpy=1.5707 0 0 -> xyz=0.10 0.09 0.05 rpy=1.5707 0 0; type continuous -> fixed
- joint front_right_wheel_joint: origin xyz=0.08 -0.09 0.05 rpy=1.5707 0 0 -> xyz=0.10 -0.09 0.05 rpy=1.5707 0 0; type continuous -> fixed
- joint rear_left_wheel_joint: origin xyz=-0.08 0.09 0.05 rpy=1.5707 0 0 -> xyz=-0.10 0.09 0.05 rpy=1.5707 0 0; type continuous -> fixed
- joint rear_right_wheel_joint: origin xyz=-0.08 -0.09 0.05 rpy=1.5707 0 0 -> xyz=-0.10 -0.09 0.05 rpy=1.5707 0 0; type continuous -> fixed
